Commit message: 完成O6接口写入，快速验证demo的完成

File: src/linker_manipulation/urdf/a7_lite_right_mesh.urdf (robot description, URDF)
Before this commit: robot a7_lite_right, 10 links, 9 joints
Links:
- added link hand_collision_proxy; collision box size=0.12 0.10 0.18; visual box size=0.12 0.10 0.18
- added link table_collision; collision box size=0.8 2.0 0.05; visual box size=0.8 2.0 0.05
Joints:
- added joint base_to_table_collision: type fixed, parent base_link, child table_collision, origin xyz=0.7 0 -0.325 rpy=0 0 0
- added joint tcp_to_hand_collision_proxy: type fixed, parent tcp_link, child hand_collision_proxy, origin xyz=0 0 -0.09 rpy=0 0 0
